Commit message: scorpio model plugin code clean-up

File: robots/Scorpio_Kin_robotiq.urdf (robot description, URDF)
Before this commit: robot Scorpio, 29 links, 28 joints
Links:
- link left_inner_finger: geometry visual mesh filename=package://gazebo_scorpio_plugin/robots/meshes/inner_finger_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
- link left_inner_knuckle: geometry visual mesh filename=package://gazebo_scorpio_plugin/robots/meshes/inner_knuckle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
- link left_outer_finger: geometry visual mesh filename=package://gazebo_scorpio_plugin/robots/meshes/outer_finger_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
- link left_outer_knuckle: geometry visual mesh filename=package://gazebo_scorpio_plugin/robots/meshes/outer_knuckle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
- link link7_end: mass 0.00000001 -> 0.00001
- link right_inner_finger: geometry visual mesh filename=package://gazebo_scorpio_plugin/robots/meshes/inner_finger_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
- link right_inner_knuckle: geometry visual mesh filename=package://gazebo_scorpio_plugin/robots/meshes/inner_knuckle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
- link right_outer_finger: geometry visual mesh filename=package://gazebo_scorpio_plugin/robots/meshes/outer_finger_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
- link right_outer_knuckle: geometry visual mesh filename=package://gazebo_scorpio_plugin/robots/meshes/outer_knuckle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
- link robotiq_85_base_link: geometry visual mesh filename=package://gazebo_scorpio_plugin/robots/meshes/robotiq_85_ba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
Joints:
- joint finger_joint: type revolute -> fixed
- joint joint10: type revolute -> continuous
- joint left_inner_finger_joint: type revolute -> fixed
- joint left_inner_knuckle_joint: type revolute -> fixed
- joint right_inner_finger_joint: type revolute -> fixed
- joint right_inner_knuckle_joint: type revolute -> fixed
- joint right_outer_knuckle_joint: type revolute -> fixed
- joint tower_mount: origin xyz=0 0 0 rpy=0 0 -1.57 -> xyz=0 0 0.5 rpy=0 0 -1.57

Commit message: create new launch file for grasping test simulation

File: robots/Scorpio_Kin_robotiq.urdf (robot description, URDF)
Before this commit: robot Scorpio, 29 links, 28 joints
Links:
- link left_inner_finger: geometry collision mesh filename=package://gazebo_scorpio_plugin/robots/meshes/inner_finger_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; visual mesh filename=package://gazebo_scorpio_plugin/robots/meshes/inner_finger_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
- link left_inner_knuckle: geometry collision mesh filename=package://gazebo_scorpio_plugin/robots/meshes/inner_knuckle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; visual mesh filename=package://gazebo_scorpio_plugin/robots/meshes/inner_knuckle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
- link left_outer_finger: geometry collision mesh filename=package://gazebo_scorpio_plugin/robots/meshes/outer_finger_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; visual mesh filename=package://gazebo_scorpio_plugin/robots/meshes/outer_finger_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
- link left_outer_knuckle: geometry collision mesh filename=package://gazebo_scorpio_plugin/robots/meshes/outer_knuckle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; visual mesh filename=package://gazebo_scorpio_plugin/robots/meshes/outer_knuckle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
- link right_inner_finger: geometry collision mesh filename=package://gazebo_scorpio_plugin/robots/meshes/inner_finger_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; visual mesh filename=package://gazebo_scorpio_plugin/robots/meshes/inner_finger_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
- link right_inner_knuckle: geometry collision mesh filename=package://gazebo_scorpio_plugin/robots/meshes/inner_knuckle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; visual mesh filename=package://gazebo_scorpio_plugin/robots/meshes/inner_knuckle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
- link right_outer_finger: geometry collision mesh filename=package://gazebo_scorpio_plugin/robots/meshes/outer_finger_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; visual mesh filename=package://gazebo_scorpio_plugin/robots/meshes/outer_finger_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
- link right_outer_knuckle: geometry collision mesh filename=package://gazebo_scorpio_plugin/robots/meshes/outer_knuckle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; visual mesh filename=package://gazebo_scorpio_plugin/robots/meshes/outer_knuckle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
- link robotiq_85_base_link: geometry collision mesh filename=package://gazebo_scorpio_plugin/robots/meshes/robotiq_85_ba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; visual mesh filename=package://gazebo_scorpio_plugin/robots/meshes/robotiq_85_ba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
