Commit message: updated to include working gripper and correct transform for scorpio_pour.world camera position - refer to updated README for changes necessary outside of this package

File: robots/Scorpio_Kin_robotiq_gripper.urdf (robot description, URDF)
Before this commit: robot Scorpio, 31 links, 30 joints
Joints:
- joint joint10: limit lower=-2.2000000 upper=1.0000000 effort=200 velocity=0 -> (none)
- joint joint11: limit lower=-3.1416 upper=3.1416 effort=200 velocity=0 -> (none); type revolute -> continuous

Commit message: Scorpio Interruption service call created

File: robots/Scorpio_Kin_robotiq_gripper.urdf (robot description, URDF)
Before this commit: robot Scorpio, 31 links, 30 joints
Joints:
- joint tower_mount: origin xyz=0 0 0.5 rpy=0 0 -1.57 -> xyz=0 0 0.5 rpy=0 0 1.57
