Commit message: further updates to README and changing mesh file syntax tomatch with README instructions

File: models/Scorpio_Kin_robotiq_gripper.urdf (robot description, URDF)
Before this commit: robot Scorpio, 29 links, 28 joints
Links:
- link left_inner_finger: geometry collision mesh filename=../../../../gazebo_scorpio_plugin/models/robotiq_2f_85/mesh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 scale=0.001 0.001 0.001; visual mesh filename=../../../../gazebo_scorpio_plugin/models/robotiq_2f_85/mesh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 scale=0.001 0.001 0.001
- link left_inner_knuckle: geometry collision mesh filename=../../../../gazebo_scorpio_plugin/models/robotiq_2f_85/mesh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 scale=0.001 0.001 0.001; visual mesh filename=../../../../gazebo_scorpio_plugin/models/robotiq_2f_85/mesh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 scale=0.001 0.001 0.001
- link left_outer_finger: geometry collision mesh filename=../../../../gazebo_scorpio_plugin/models/robotiq_2f_85/mesh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 scale=0.001 0.001 0.001; visual mesh filename=../../../../gazebo_scorpio_plugin/models/robotiq_2f_85/mesh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 scale=0.001 0.001 0.001
- link left_outer_knuckle: geometry collision mesh filename=../../../../gazebo_scorpio_plugin/models/robotiq_2f_85/mesh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 scale=0.001 0.001 0.001; visual mesh filename=../../../../gazebo_scorpio_plugin/models/robotiq_2f_85/mesh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 scale=0.001 0.001 0.001
- link link1: geometry visual mesh filename=../../../../gazebo_scorpio_plugin/models/robots/meshes/scor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
- link link2: geometry visual mesh filename=../../../../gazebo_scorpio_plugin/models/robots/meshes/para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
- link link3: geometry visual mesh filename=../../../../gazebo_scorpio_plugin/models/robots/meshes/para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
- link link4: geometry visual mesh filename=../../../../gazebo_scorpio_plugin/models/robots/meshes/para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
- link link5: geometry visual mesh filename=../../../../gazebo_scorpio_plugin/models/robots/meshes/scor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
- link link6: geometry visual mesh filename=../../../../gazebo_scorpio_plugin/models/robots/meshes/para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
- link link7: geometry visual mesh filename=../../../../gazebo_scorpio_plugin/models/robots/meshes/para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
- link link8: geometry visual mesh filename=../../../../gazebo_scorpio_plugin/models/robots/meshes/para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
- link link9: geometry visual mesh filename=../../../../gazebo_scorpio_plugin/models/robots/meshes/scor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
- link right_inner_finger: geometry collision mesh filename=../../../../gazebo_scorpio_plugin/models/robotiq_2f_85/mesh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 scale=0.001 0.001 0.001; visual mesh filename=../../../../gazebo_scorpio_plugin/models/robotiq_2f_85/mesh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 scale=0.001 0.001 0.001
- link right_inner_knuckle: geometry collision mesh filename=../../../../gazebo_scorpio_plugin/models/robotiq_2f_85/mesh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 scale=0.001 0.001 0.001; visual mesh filename=../../../../gazebo_scorpio_plugin/models/robotiq_2f_85/mesh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 scale=0.001 0.001 0.001
- link right_outer_finger: geometry collision mesh filename=../../../../gazebo_scorpio_plugin/models/robotiq_2f_85/mesh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 scale=0.001 0.001 0.001; visual mesh filename=../../../../gazebo_scorpio_plugin/models/robotiq_2f_85/mesh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 scale=0.001 0.001 0.001
- link right_outer_knuckle: geometry collision mesh filename=../../../../gazebo_scorpio_plugin/models/robotiq_2f_85/mesh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 scale=0.001 0.001 0.001; visual mesh filename=../../../../gazebo_scorpio_plugin/models/robotiq_2f_85/mesh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 scale=0.001 0.001 0.001
- link robotiq_85_base_link: geometry collision mesh filename=../../../../gazebo_scorpio_plugin/models/robotiq_2f_85/mesh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; visual mesh filename=../../../../gazebo_scorpio_plugin/models/robotiq_2f_85/mesh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
- link scorpio_ground: geometry visual mesh filename=../../../../gazebo_scorpio_plugin/models/robots/meshes/scor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
- link scorpio_wrist_pitch: geometry visual mesh filename=../../../../gazebo_scorpio_plugin/models/robots/meshes/scor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

File: models/robots/Scorpio_Kin_robotiq.urdf (robot description, URDF)
Before this commit: robot Scorpio, 29 links, 28 joints
Links:
- link left_inner_finger: geometry collision mesh filename=package://gazebo_scorpio_plugin/models/robots/meshes/inner_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; visual mesh filename=package://gazebo_scorpio_plugin/models/robots/meshes/inner_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
- link left_inner_knuckle: geometry collision mesh filename=package://gazebo_scorpio_plugin/models/robots/meshes/inner_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; visual mesh filename=package://gazebo_scorpio_plugin/models/robots/meshes/inner_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
- link left_outer_finger: geometry collision mesh filename=package://gazebo_scorpio_plugin/models/robots/meshes/outer_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; visual mesh filename=package://gazebo_scorpio_plugin/models/robots/meshes/outer_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
- link left_outer_knuckle: geometry collision mesh filename=package://gazebo_scorpio_plugin/models/robots/meshes/outer_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; visual mesh filename=package://gazebo_scorpio_plugin/models/robots/meshes/outer_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
- link link1: geometry visual mesh filename=package://gazebo_scorpio_plugin/models/robots/meshes/scorpi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
- link link2: geometry visual mesh filename=package://gazebo_scorpio_plugin/models/robots/meshes/parall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
- link link3: geometry visual mesh filename=package://gazebo_scorpio_plugin/models/robots/meshes/parall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
- link link4: geometry visual mesh filename=package://gazebo_scorpio_plugin/models/robots/meshes/parall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
- link link5: geometry visual mesh filename=package://gazebo_scorpio_plugin/models/robots/meshes/scorpi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
- link link6: geometry visual mesh filename=package://gazebo_scorpio_plugin/models/robots/meshes/parall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
- link link7: geometry visual mesh filename=package://gazebo_scorpio_plugin/models/robots/meshes/parall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
- link link8: geometry visual mesh filename=package://gazebo_scorpio_plugin/models/robots/meshes/parall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
- link link9: geometry visual mesh filename=package://gazebo_scorpio_plugin/models/robots/meshes/scorpi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
- link right_inner_finger: geometry collision mesh filename=package://gazebo_scorpio_plugin/models/robots/meshes/inner_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; visual mesh filename=package://gazebo_scorpio_plugin/models/robots/meshes/inner_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
- link right_inner_knuckle: geometry collision mesh filename=package://gazebo_scorpio_plugin/models/robots/meshes/inner_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; visual mesh filename=package://gazebo_scorpio_plugin/models/robots/meshes/inner_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
- link right_outer_finger: geometry collision mesh filename=package://gazebo_scorpio_plugin/models/robots/meshes/outer_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; visual mesh filename=package://gazebo_scorpio_plugin/models/robots/meshes/outer_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
- link right_outer_knuckle: geometry collision mesh filename=package://gazebo_scorpio_plugin/models/robots/meshes/outer_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; visual mesh filename=package://gazebo_scorpio_plugin/models/robots/meshes/outer_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
- link robotiq_85_base_link: geometry collision mesh filename=package://gazebo_scorpio_plugin/models/robots/meshes/roboti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; visual mesh filename=package://gazebo_scorpio_plugin/models/robots/meshes/roboti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
- link scorpio_ground: geometry visual mesh filename=package://gazebo_scorpio_plugin/models/robots/meshes/scorpi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
- link scorpio_wrist_pitch: geometry visual mesh filename=package://gazebo_scorpio_plugin/models/robots/meshes/scorpi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

File: models/robots/Scorpio_Kin_robotiq_gripper.urdf (robot description, URDF)
Before this commit: robot Scorpio, 31 links, 30 joints
Links:
- link left_inner_finger: geometry collision mesh filename=model://robotiq_2f_85/meshes/collision/robotiq_arg2f_85_inn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 scale=0.001 0.001 0.001; visual mesh filename=model://robotiq_2f_85/meshes/visual/robotiq_arg2f_85_inner_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 scale=0.001 0.001 0.001
- link left_inner_knuckle: geometry collision mesh filename=model://robotiq_2f_85/meshes/collision/robotiq_arg2f_85_inn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 scale=0.001 0.001 0.001; visual mesh filename=model://robotiq_2f_85/meshes/visual/robotiq_arg2f_85_inner_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 scale=0.001 0.001 0.001
- link left_outer_finger: geometry collision mesh filename=model://robotiq_2f_85/meshes/collision/robotiq_arg2f_85_out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 scale=0.001 0.001 0.001; visual mesh filename=model://robotiq_2f_85/meshes/visual/robotiq_arg2f_85_outer_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 scale=0.001 0.001 0.001
- link left_outer_knuckle: geometry collision mesh filename=model://robotiq_2f_85/meshes/collision/robotiq_arg2f_85_out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 scale=0.001 0.001 0.001; visual mesh filename=model://robotiq_2f_85/meshes/visual/robotiq_arg2f_85_outer_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 scale=0.001 0.001 0.001
- link link1: geometry visual mesh filename=model://robots/meshes/scorpio_yaw1_hull.dae
- link link2: geometry visual mesh filename=model://robots/meshes/parallel__scorpio_elev1__l3_hull.dae
- link link3: geometry visual mesh filename=model://robots/meshes/parallel__scorpio_elev1__l2_hull.dae
- link link4: geometry visual mesh filename=model://robots/meshes/parallel__scorpio_elev1__l1_hull.dae
- link link5: geometry visual mesh filename=model://robots/meshes/scorpio_yaw2_hull.dae
- link link6: geometry visual mesh filename=model://robots/meshes/parallel__scorpio_elev2__l3_hull.dae
- link link7: geometry visual mesh filename=model://robots/meshes/parallel__scorpio_elev2__l2_hull.dae
- link link8: geometry visual mesh filename=model://robots/meshes/parallel__scorpio_elev2__l1_hull.dae
- link link9: geometry visual mesh filename=model://robots/meshes/scorpio_wrist_skewed_hull.dae
- link right_inner_finger: geometry collision mesh filename=model://robotiq_2f_85/meshes/collision/robotiq_arg2f_85_inn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 scale=0.001 0.001 0.001; visual mesh filename=model://robotiq_2f_85/meshes/visual/robotiq_arg2f_85_inner_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 scale=0.001 0.001 0.001
- link right_inner_knuckle: geometry collision mesh filename=model://robotiq_2f_85/meshes/collision/robotiq_arg2f_85_inn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 scale=0.001 0.001 0.001; visual mesh filename=model://robotiq_2f_85/meshes/visual/robotiq_arg2f_85_inner_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 scale=0.001 0.001 0.001
- link right_outer_finger: geometry collision mesh filename=model://robotiq_2f_85/meshes/collision/robotiq_arg2f_85_out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 scale=0.001 0.001 0.001; visual mesh filename=model://robotiq_2f_85/meshes/visual/robotiq_arg2f_85_outer_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 scale=0.001 0.001 0.001
- link right_outer_knuckle: geometry collision mesh filename=model://robotiq_2f_85/meshes/collision/robotiq_arg2f_85_out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 scale=0.001 0.001 0.001; visual mesh filename=model://robotiq_2f_85/meshes/visual/robotiq_arg2f_85_outer_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 scale=0.001 0.001 0.001
- link robotiq_arg2f_base_link: geometry collision mesh filename=model://robotiq_2f_85/meshes/collision/robotiq_arg2f_base_l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; visual mesh filename=model://robotiq_2f_85/meshes/collision/robotiq_arg2f_base_l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
- link scorpio_ground: geometry visual mesh filename=model://robots/meshes/scorpio_ground_hull.dae
- link scorpio_wrist_pitch: geometry visual mesh filename=model://robots/meshes/scorpio_wrist_pitch_hull.dae

File: models/robots/Scorpio_Kin_robotiq_new.urdf (robot description, URDF)
Before this commit: robot Scorpio, 29 links, 28 joints
Links:
- link left_inner_finger: geometry collision mesh filename=package://gazebo_scorpio_plugin/models/robots/meshes/inner_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; visual mesh filename=package://gazebo_scorpio_plugin/models/robots/meshes/inner_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
- link left_inner_knuckle: geometry collision mesh filename=package://gazebo_scorpio_plugin/models/robots/meshes/inner_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; visual mesh filename=package://gazebo_scorpio_plugin/models/robots/meshes/inner_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
- link left_outer_finger: geometry collision mesh filename=package://gazebo_scorpio_plugin/models/robots/meshes/outer_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; visual mesh filename=package://gazebo_scorpio_plugin/models/robots/meshes/outer_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
- link left_outer_knuckle: geometry collision mesh filename=package://gazebo_scorpio_plugin/models/robots/meshes/outer_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; visual mesh filename=package://gazebo_scorpio_plugin/models/robots/meshes/outer_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
- link link1: geometry visual mesh filename=package://gazebo_scorpio_plugin/models/robots/meshes/scorpi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
- link link2: geometry visual mesh filename=package://gazebo_scorpio_plugin/models/robots/meshes/parall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
- link link3: geometry visual mesh filename=package://gazebo_scorpio_plugin/models/robots/meshes/parall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
- link link4: geometry visual mesh filename=package://gazebo_scorpio_plugin/models/robots/meshes/parall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
- link link5: geometry visual mesh filename=package://gazebo_scorpio_plugin/models/robots/meshes/scorpi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
- link link6: geometry visual mesh filename=package://gazebo_scorpio_plugin/models/robots/meshes/parall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
- link link7: geometry visual mesh filename=package://gazebo_scorpio_plugin/models/robots/meshes/parall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
- link link8: geometry visual mesh filename=package://gazebo_scorpio_plugin/models/robots/meshes/parall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
- link link9: geometry visual mesh filename=package://gazebo_scorpio_plugin/models/robots/meshes/scorpi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
- link right_inner_finger: geometry collision mesh filename=package://gazebo_scorpio_plugin/models/robots/meshes/inner_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; visual mesh filename=package://gazebo_scorpio_plugin/models/robots/meshes/inner_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
- link right_inner_knuckle: geometry collision mesh filename=package://gazebo_scorpio_plugin/models/robots/meshes/inner_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; visual mesh filename=package://gazebo_scorpio_plugin/models/robots/meshes/inner_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
- link right_outer_finger: geometry collision mesh filename=package://gazebo_scorpio_plugin/models/robots/meshes/outer_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; visual mesh filename=package://gazebo_scorpio_plugin/models/robots/meshes/outer_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
- link right_outer_knuckle: geometry collision mesh filename=package://gazebo_scorpio_plugin/models/robots/meshes/outer_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; visual mesh filename=package://gazebo_scorpio_plugin/models/robots/meshes/outer_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
- link robotiq_85_base_link: geometry collision mesh filename=package://gazebo_scorpio_plugin/models/robots/meshes/roboti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; visual mesh filename=package://gazebo_scorpio_plugin/models/robots/meshes/roboti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
- link scorpio_ground: geometry visual mesh filename=package://gazebo_scorpio_plugin/models/robots/meshes/scorpi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
- link scorpio_wrist_pitch: geometry visual mesh filename=package://gazebo_scorpio_plugin/models/robots/meshes/scorpi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
